File: Spring_2025/NathanHuang_Sp25_1/NathanHuang_Sp25_1.kicad_sch (KiCad schematic)
At the start: 10 parts, among them J1 Barrel_Jack, M1 Motor_Servo, M2 Motor_Servo, M3 Motor_Servo, M4 Motor_Servo, M5 Motor_Servo, M6 Motor_Servo, M7 Stepper_Motor_bipolar, U1 ESP32-DEVKITC-32UE

Commit message: Schematic Done
Parts:
- added C1: 22u, Capacitor_THT:CP_Radial_Tantal_D5.0mm_P2.50mm, symbol Device:C
- added U2: LM2596_BUCK_CONVERTER, Library:LM2596_BUCK_CONVERTER, symbol Library:LM2596_BUCK_CONVERTER
- J1: footprint (none) -> Connector_BarrelJack:BarrelJack_SwitchcraftConxall_RAPC10U_Horizontal
- M1, M2, M3, M4, M5, M6: footprint (none) -> Connector_PinHeader_1.00mm:PinHeader_1x03_P1.00mm_Horizontal
- M7: footprint (none) -> Connector_PinHeader_1.00mm:PinHeader_1x04_P1.00mm_Horizontal
- U1: footprint ESP32-DEVKITC-32UE:ESPRESSIF_ESP32-DEVKITC-32UE -> Library:ESP32-DEVKITC-32UE
Connections:
- net +12V: now also J1.1, C1.1, U2.1 (Vin)
- net +5V: no longer U1.2 (EN)
- net DIR_PIN: now also U1.35 (15)
- net GND: now also J1.2, C1.2, U2.2 (GND), U2.3 (GND)
- net STEP_PIN: now also U1.12 (14)
- net 7.2V: now reaches M4.2 (+)
- net 7.2V: now also M1.2 (+), M2.2 (+), M3.2 (+), M5.2 (+), M6.2 (+), U2.4 (Vout)
- no-connect marks 14 -> 29
Other:
- note added: "POWER"
- note added: "PWR FLAGS"

Commit message: Finished PCB, Ready for Print
Parts:
- added H1, H2, H3, H4: MountingHole, MountingHole:MountingHole_2.1mm, symbol Mechanical:MountingHole
Connections:
- net DIR_PIN: now also U1.6 (35); no longer U1.35 (15)
- net INDEX: now also U1.25 (21); no longer U1.33 (0)
- net MIDDLE: now also U1.28 (18); no longer U1.34 (2)
- net PINKIE: now also U1.34 (2); no longer U1.29 (5)
- net RING: now also U1.31 (16); no longer U1.32 (4)
- net STEP_PIN: now also U1.7 (32); no longer U1.12 (14)
- net THUMB_1: now also U1.21 (23); no longer U1.13 (12)
- net THUMB_2: now also U1.22; no longer U1.15 (13)
- net +3V3: now reaches U1.1 (3V3)
- net +3V3: now also A1.2 (VDD)
- net at M7.1: now also A1.6 (2B); no longer A1.3 (1B)
- net at M7.2 (-): now also A1.5 (2A); no longer A1.4 (1A)
- net at M7.3: now also A1.4 (1A); no longer A1.5 (2A)
- net at M7.4: now also A1.3 (1B); no longer A1.6 (2B)
- net +5V: no longer names the net of U1.19 (5V)
- net +5V: no longer A1.2 (VDD)
Other:
- moved on the sheet: M7

Commit message: PCB Updates
Parts:
- removed U1: ESP32-DEVKITC-32UE, Library:ESP32-DEVKITC-32UE, symbol Library:ESP32-DEVKITC-32UE
- added Encoder1: ~, Connector_PinHeader_2.54mm:PinHeader_1x04_P2.54mm_Horizontal, symbol Library:Encoder
- added SW1, SW2: SW_Push, Connector_PinHeader_2.54mm:PinHeader_1x02_P2.54mm_Horizontal, symbol Switch:SW_Push
- added U1: ESP32-WROOM-32, RF_Module:ESP32-WROOM-32, symbol RF_Module:ESP32-WROOM-32
- C1: footprint Capacitor_THT:CP_Radial_Tantal_D5.0mm_P2.50mm -> Capacitor_THT:CP_Radial_D4.0mm_P1.50mm
- H1, H2, H3, H4: footprint MountingHole:MountingHole_2.1mm -> MountingHole:MountingHole_5.3mm_M5
- M1, M2, M3, M4, M5, M6: footprint Connector_PinHeader_1.00mm:PinHeader_1x03_P1.00mm_Horizontal -> Connector_PinHeader_2.54mm:PinHeader_1x03_P2.54mm_Horizontal
- M7: footprint Connector_PinHeader_1.00mm:PinHeader_1x04_P1.00mm_Horizontal -> Connector_PinHeader_2.54mm:PinHeader_1x04_P2.54mm_Horizontal
Connections:
- net +3V3: now also Encoder1. (VCC), SW1.2, SW2.2, U1.2 (VDD)
- net DIR_PIN: now also U1.36 (IO22)
- net GND: now also Encoder1. (VCC), U1.1 (GND), U1.15 (GND), U1.38 (GND), U1.39 (GND)
- net INDEX: now also U1.28 (IO17)
- net MIDDLE: now also U1.27 (IO16)
- net PINKIE: now also U1.14 (IO12)
- net RING: now also U1.23 (IO15)
- net STEP_PIN: now also U1.33 (IO21)
- net THUMB_1: now also U1.31 (IO19)
- net THUMB_2: now also U1.30 (IO18)
- new net: SW1.1, U1.25 (IO0)
- new net: SW2.1, U1.26 (IO4)
- new net CW: Encoder1. (VCC), U1.16 (IO13)
- new net DT: Encoder1. (VCC), U1.13 (IO14)
- no-connect marks 29 -> 23
Other:
- note added: "ENCODER"
- note added: "MOUNTING HOLES"
- moved on the sheet: H1, H2, H3, H4

Commit message: 4/4 Changes
Connections:
- net +3V3: now also Encoder1.3 (VCC); no longer Encoder1. (VCC)
- net CW: now also Encoder1.2 (CW); no longer Encoder1. (VCC)
- net DT: now also Encoder1.1 (DT); no longer Encoder1. (VCC)
- net GND: now also Encoder1.4 (GND); no longer Encoder1. (VCC)
Changed lines of the file:
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@@
 	(wire
 		(pts
+			(xy 186.69 148.59) (xy 184.15 148.59)
+		)
+		(stroke
+			(width 0)
+			(type default)
+		)
+	)
+	(wire
+		(pts
 			(xy 187.96 83.82) (xy 190.5 83.82)
 		)
@@
 	(wire
 		(pts
+			(xy 186.69 146.05) (xy 184.15 146.05)
+		)
+		(stroke
+			(width 0)
+			(type default)
+		)
+	)
+	(wire
+		(pts
 			(xy 106.68 135.89) (xy 119.38 135.89)
 		)
@@
 	(wire
 		(pts
-			(xy 180.34 140.97) (xy 184.15 140.97)
+			(xy 180.34 140.97) (xy 186.69 140.97)
 		)
 		(stroke
@@
 	(wire
 		(pts
-			(xy 180.34 143.51) (xy 184.15 143.51)
+			(xy 180.34 143.51) (xy 186.69 143.51)
 		)
 		(stroke
@@
 	(symbol
 		(lib_id "Library:Encoder")
-		(at 181.61 144.78 0)
+		(at 184.15 144.78 0)
 		(unit 1)
 		(exclude_from_sim no)
@@
 		(fields_autoplaced yes)
 		(property "Reference" "Encoder1"
-			(at 194.31 144.1449 0)
+			(at 196.85 144.1449 0)
 			(effects
 				(font
@@
 		)
 		(property "Value" "~"
-			(at 194.31 146.05 0)
+			(at 196.85 146.05 0)
 			(effects
 				(font
@@
 		)
 		(property "Footprint" "Connector_PinHeader_2.54mm:PinHeader_1x04_P2.54mm_Horizontal"
-			(at 181.61 144.78 0)
+			(at 185.928 152.908 0)
 			(effects
 				(font
@@
 		)
 		(property "Datasheet" ""
-			(at 181.61 144.78 0)
+			(at 184.15 144.78 0)
 			(effects
 				(font
@@
 		)
 		(property "Description" ""
-			(at 181.61 144.78 0)
+			(at 184.15 144.78 0)
 			(effects
 				(font
@@
 			)
 		)
-		(pin ""
+		(pin "1"
 		)
-		(pin ""
+		(pin "4"
 		)
-		(pin ""
+		(pin "3"
 		)
-		(pin ""
+		(pin "2"
 		)
 		(instances

Commit message: Found Footprint
New to find new schematic for 30 pin
Parts:
- Encoder1: footprint Connector_PinHeader_2.54mm:PinHeader_1x04_P2.54mm_Horizontal -> Connector_PinHeader_2.54mm:PinHeader_1x04_P2.54mm_Vertical
- M1, M2, M3, M4, M5, M6: footprint Connector_PinHeader_2.54mm:PinHeader_1x03_P2.54mm_Horizontal -> Connector_PinHeader_2.54mm:PinHeader_1x03_P2.54mm_Vertical
- M7: footprint Connector_PinHeader_2.54mm:PinHeader_1x04_P2.54mm_Horizontal -> Connector_PinHeader_2.54mm:PinHeader_1x03_P2.54mm_Vertical
- SW1, SW2: footprint Connector_PinHeader_2.54mm:PinHeader_1x02_P2.54mm_Horizontal -> Connector_PinHeader_2.54mm:PinHeader_1x02_P2.54mm_Vertical
- U1: footprint RF_Module:ESP32-WROOM-32 -> Library:ESP32-WROOM-32
Other:
- note added: "PADs 31-36 DNE"
Changed lines of the file:
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@@
 	)
 	(rectangle
-		(start 12.7 29.21)
+		(start 12.7 25.4)
 		(end 86.36 123.19)
 		(stroke
@@
 	(text "MICROCONTROLLER"
 		(exclude_from_sim no)
-		(at 38.862 27.94 0)
+		(at 22.86 22.86 0)
 		(effects
 			(font
@@
 		)
 	)
+	(text "PADs 31-36 DNE"
+		(exclude_from_sim no)
+		(at -6.096 54.61 0)
+		(effects
+			(font
+				(size 1.27 1.27)
+			)
+		)
+	)
 	(label "MIDDLE"
 		(at 120.65 54.61 180)
@@
 			)
 		)
-		(property "Footprint" "Connector_PinHeader_2.54mm:PinHeader_1x03_P2.54mm_Horizontal"
+		(property "Footprint" "Connector_PinHeader_2.54mm:PinHeader_1x03_P2.54mm_Vertical"
 			(at 130.81 84.836 0)
 			(effects
@@
 			)
 		)
-		(property "Footprint" "Connector_PinHeader_2.54mm:PinHeader_1x03_P2.54mm_Horizontal"
+		(property "Footprint" "Connector_PinHeader_2.54mm:PinHeader_1x03_P2.54mm_Vertical"
 			(at 130.81 73.406 0)
 			(effects
@@
 			)
 		)
-		(property "Footprint" "Connector_PinHeader_2.54mm:PinHeader_1x04_P2.54mm_Horizontal"
+		(property "Footprint" "Connector_PinHeader_2.54mm:PinHeader_1x03_P2.54mm_Vertical"
 			(at 157.734 143.256 0)
 			(effects
@@
 			)
 		)
-		(property "Footprint" "Connector_PinHeader_2.54mm:PinHeader_1x02_P2.54mm_Horizontal"
+		(property "Footprint" "Connector_PinHeader_2.54mm:PinHeader_1x02_P2.54mm_Vertical"
 			(at 60.96 36.83 0)
 			(effects
@@
 			)
 		)
-		(property "Footprint" "Connector_PinHeader_2.54mm:PinHeader_1x03_P2.54mm_Horizontal"
+		(property "Footprint" "Connector_PinHeader_2.54mm:PinHeader_1x03_P2.54mm_Vertical"
 			(at 130.81 107.696 0)
 			(effects
@@
 			)
 		)
-		(property "Footprint" "Connector_PinHeader_2.54mm:PinHeader_1x02_P2.54mm_Horizontal"
+		(property "Footprint" "Connector_PinHeader_2.54mm:PinHeader_1x02_P2.54mm_Vertical"
 			(at 60.96 46.99 0)
 			(effects
@@
 			)
 		)
-		(property "Footprint" "Connector_PinHeader_2.54mm:PinHeader_1x03_P2.54mm_Horizontal"
+		(property "Footprint" "Connector_PinHeader_2.54mm:PinHeader_1x03_P2.54mm_Vertical"
 			(at 130.81 50.546 0)
 			(effects
@@
 			)
 		)
-		(property "Footprint" "Connector_PinHeader_2.54mm:PinHeader_1x03_P2.54mm_Horizontal"
+		(property "Footprint" "Connector_PinHeader_2.54mm:PinHeader_1x03_P2.54mm_Vertical"
 			(at 130.81 96.266 0)
 			(effects
@@
 		(on_board yes)
 		(dnp no)
-		(fields_autoplaced yes)
 		(property "Reference" "U1"
 			(at 36.4841 34.29 0)
@@
 		)
 		(property "Value" "ESP32-WROOM-32"
-			(at 36.4841 36.83 0)
+			(at 25.908 28.702 0)
 			(effects
 				(font
@@
 			)
 		)
-		(property "Footprint" "RF_Module:ESP32-WROOM-32"
+		(property "Footprint" "Library:ESP32-WROOM-32"
 			(at 34.29 110.49 0)
 			(effects
@@
 			)
 		)
-		(property "Footprint" "Connector_PinHeader_2.54mm:PinHeader_1x03_P2.54mm_Horizontal"
+		(property "Footprint" "Connector_PinHeader_2.54mm:PinHeader_1x03_P2.54mm_Vertical"
 			(at 130.81 61.976 0)
 			(effects
@@
 			)
 		)
-		(property "Footprint" "Connector_PinHeader_2.54mm:PinHeader_1x04_P2.54mm_Horizontal"
+		(property "Footprint" "Connector_PinHeader_2.54mm:PinHeader_1x04_P2.54mm_Vertical"
 			(at 185.928 152.908 0)
 			(effects

Commit message: Changes
Parts:
- removed U1: ESP32-WROOM-32, Library:ESP32-WROOM-32, symbol RF_Module:ESP32-WROOM-32
- added U3: ESP32-WROOM-32, symbol Library:ESP32-WROOM-32
Changed lines of the file:
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@@
-	)
-	(symbol
-		(lib_id "RF_Module:ESP32-WROOM-32")
-		(at 34.29 72.39 0)
-		(unit 1)
-		(exclude_from_sim no)
-		(in_bom yes)
-		(on_board yes)
-		(dnp no)
-		(property "Reference" "U1"
-			(at 36.4841 34.29 0)
-			(effects
-				(font
-					(size 1.27 1.27)
-				)
-				(justify left)
-			)
-		)
-		(property "Value" "ESP32-WROOM-32"
-			(at 25.908 28.702 0)
-			(effects
-				(font
-					(size 1.27 1.27)
-				)
-				(justify left)
-			)
-		)
-		(property "Footprint" "Library:ESP32-WROOM-32"
-			(at 34.29 110.49 0)
-			(effects
-				(font
-					(size 1.27 1.27)
-				)
-				(hide yes)
-			)
-		)
-		(property "Datasheet" "https://www.espressif.com/sites/default/files/documentation/esp32-wroom-32_datasheet_en.pdf"
-			(at 26.67 71.12 0)
-			(effects
-				(font
-					(size 1.27 1.27)
-				)
-				(hide yes)
-			)
-		)
-		(property "Description" "RF Module, ESP32-D0WDQ6 SoC, Wi-Fi 802.11b/g/n, Bluetooth, BLE, 32-bit, 2.7-3.6V, onboard antenna, SMD"
-			(at 34.29 72.39 0)
-			(effects
-				(font
-					(size 1.27 1.27)
-				)
-				(hide yes)
-			)
-		)
-		(pin "7"
-		)
-		(pin "8"
-		)
-		(pin "34"
-		)
-		(pin "13"
-		)
-		(pin "15"
-		)
-		(pin "3"
-		)
-		(pin "12"
-		)
-		(pin "21"
-		)
-		(pin "24"
-		)
-		(pin "1"
-		)
-		(pin "2"
-		)
-		(pin "26"
-		)
-		(pin "11"
-		)
-		(pin "22"
-		)
-		(pin "27"
-		)
-		(pin "20"
-		)
-		(pin "31"
-		)
-		(pin "19"
-		)
-		(pin "23"
-		)
-		(pin "36"
-		)
-		(pin "4"
-		)
-		(pin "5"
-		)
-		(pin "17"
-		)
-		(pin "9"
-		)
-		(pin "39"
-		)
-		(pin "35"
-		)
-		(pin "25"
-		)
-		(pin "37"
-		)
-		(pin "6"
-		)
-		(pin "38"
-		)
-		(pin "10"
-		)
-		(pin "28"
-		)
-		(pin "14"
-		)
-		(pin "29"
-		)
-		(pin "16"
-		)
-		(pin "18"
-		)
-		(pin "30"
-		)
-		(pin "32"
-		)
-		(pin "33"
-		)
-		(instances
-			(project ""
-				(path "/ab2041eb-320e-4b4d-9636-e8f50e038a2e"
-					(reference "U1")
-					(unit 1)
-				)
-			)
-		)
 	)
 	(symbol
@@
 					(unit 1)
 				)
+			)
+		)
+	)
+	(symbol
+		(lib_id "Library:ESP32-WROOM-32")
+		(at 34.29 76.2 0)
+		(unit 1)
+		(exclude_from_sim no)
+		(in_bom yes)
+		(on_board yes)
+		(dnp no)
+		(fields_autoplaced yes)
+		(property "Reference" "U3"
+			(at 34.29 52.07 0)
+			(effects
+				(font
+					(size 1.27 1.27)
+				)
+			)
+		)
+		(property "Value" "ESP32-WROOM-32"
+			(at 34.29 54.61 0)
+			(effects
+				(font
+					(size 1.27 1.27)
+				)
+			)
+		)
+		(property "Footprint" ""
+			(at 40.64 76.2 0)
+			(effects
+				(font
+					(size 1.27 1.27)
+				)
+			)
+		)
+		(property "Datasheet" ""
+			(at 40.64 76.2 0)
+			(effects
+				(font
+					(size 1.27 1.27)
+				)
+			)
+		)
+		(property "Description" "NodeMCU 0.9"
+			(at 34.29 76.2 0)
+			(effects
+				(font
+					(size 1.27 1.27)
+				)
+				(hide yes)
+			)
+		)
+		(pin "13"
+		)
+		(pin "18"
+		)
+		(pin "2"
+		)
+		(pin "21"
+		)
+		(pin "23"
+		)
+		(pin "24"
+		)
+		(pin "26"
+		)
+		(pin "27"
+		)
+		(pin "29"
+		)
+		(pin "22"
+		)
+		(pin "19"
+		)
+		(pin "10"
+		)
+		(pin "20"
+		)
+		(pin "25"
+		)
+		(pin "3"
+		)
+		(pin "4"
+		)
+		(pin "15"
+		)
+		(pin "28"
+		)
+		(pin "30"
+		)
+		(pin "1"
+		)
+		(pin "12"
+		)
+		(pin "17"
+		)
+		(pin "11"
+		)
+		(pin "14"
+		)
+		(pin "16"
+		)
+		(pin "7"
+		)
+		(pin "9"
+		)
+		(pin "5"
+		)
+		(pin "6"
+		)
+		(pin "8"
+		)
+		(instances
+			(project ""
+				(path "/ab2041eb-320e-4b4d-9636-e8f50e038a2e"
+					(reference "U3")
+					(unit 1)
+				)

Commit message: Overwrite Changes
Connections:
- net +3V3: now also U3.30 (3V3)
- net CW: now also U3.6 (G32)
- net DIR_PIN: now also U3.28 (G15)
- net DT: now also U3.5 (G35)
- net GND: now also U3.14 (GND), U3.29 (GND)
- net INDEX: now also U3.21 (G19)
- net MIDDLE: now also U3.20 (G21)
- net PINKIE: now also U3.17 (G22)
- net RING: now also U3.4 (G34)
- net STEP_PIN: now also U3.27 (G2)
- net THUMB_1: now also U3.26 (G4)
- net THUMB_2: now also U3.22 (G18)
- net at SW1.1: now also U3.11 (G14)
- net at SW2.1: now also U3.8 (G25)
- no-connect marks 23 -> 17
Other:
- moved on the sheet: SW1, SW2, U3
