File: Spring_2025/NathanHuang_Sp25_1/NathanHuang_Sp25_1.kicad_sch (KiCad schematic)
At the start: 19 parts, among them J1 Barrel_Jack, M1 Motor_Servo, M2 Motor_Servo, M3 Motor_Servo, M4 Motor_Servo, M5 Motor_Servo, M6 Motor_Servo, M7 Stepper_Motor_bipolar, SW1 SW_Push, SW2 SW_Push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

Commit message: Updated PCB schematic
Connections:
- net PINKY is gone; now on net PINKIE: M6.1 (PWM)
- net +3V3: now also Encoder1.3 (VCC); no longer Encoder1.2 (VCC)
- net CW: now also Encoder1.2 (CW), U3.13 (G13); no longer Encoder1.3 (CW), U3.6 (G32)
- net DIR_PIN: now also U3.4 (G34); no longer U3.28 (G15)
- net DT: now also Encoder1.1 (DT), U3.12 (G12); no longer Encoder1.4 (DT), U3.5 (G35)
- net GND: now also Encoder1.4 (GND); no longer Encoder1.1 (GND)
- net INDEX: now also U3.20 (G21); no longer U3.21 (G19)
- net MIDDLE: now also U3.21 (G19); no longer U3.20 (G21)
- net PINKIE: now also U3.26 (G4); no longer U3.17 (G22)
- net RING: now also U3.22 (G18); no longer U3.4 (G34)
- net STEP_PIN: now also U3.5 (G35); no longer U3.27 (G2)
- net THUMB_1: now also U3.16 (G23); no longer U3.26 (G4)
- net THUMB_2: now also U3.17 (G22); no longer U3.22 (G18)
- net at U3.11 (G14): no longer SW1.1
- net at U3.8 (G25): no longer SW2.1
- new net SW1: SW1.1, U3.27 (G2)
- new net SW2: SW2.1, U3.28 (G15)
Other:
- moved on the sheet: H4, SW2
