File: Spring_2025/NathanHuang_Sp25_1/NathanHuang_Sp25_1.kicad_sch (KiCad schematic)
At the start: 19 parts, among them J1 Barrel_Jack, M1 Motor_Servo, M2 Motor_Servo, M3 Motor_Servo, M4 Motor_Servo, M5 Motor_Servo, M6 Motor_Servo, M7 Stepper_Motor_bipolar, SW1 SW_Push, SW2 SW_Push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

Commit message: Changes
Parts:
- M7: footprint Connector_PinHeader_2.54mm:PinHeader_1x03_P2.54mm_Vertical -> Connector_PinHeader_2.54mm:PinHeader_1x04_P2.54mm_Vertical
- U3: footprint (none) -> Library:ESP32-WROOM-32
Connections:
- net +3V3: now also Encoder1.2 (VCC); no longer Encoder1.3 (VCC)
- net CW: now also Encoder1.3 (CW); no longer Encoder1.2 (CW)
- net DT: now also Encoder1.4 (DT); no longer Encoder1.1 (DT)
- net GND: now also Encoder1.1 (GND); no longer Encoder1.4 (GND)
- net INDEX: now also M3.1 (PWM); no longer M1.1 (PWM)
- net MIDDLE: now also M4.1 (PWM); no longer M2.1 (PWM)
- net PINKIE: no longer M4.1 (PWM)
- net RING: now also M5.1 (PWM); no longer M3.1 (PWM)
- net THUMB_1: now also M1.1 (PWM); no longer M5.1 (PWM)
- net THUMB_2: now also M2.1 (PWM); no longer M6.1 (PWM)
- new net PINKY: M6.1 (PWM)
Other:
- moved on the sheet: H4
Changed lines of the file:
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@@
 	(wire
 		(pts
-			(xy 186.69 148.59) (xy 184.15 148.59)
+			(xy 186.69 140.97) (xy 184.15 140.97)
 		)
 		(stroke
@@
 	(wire
 		(pts
-			(xy 186.69 146.05) (xy 184.15 146.05)
+			(xy 186.69 143.51) (xy 184.15 143.51)
 		)
 		(stroke
@@
 	(wire
 		(pts
-			(xy 180.34 140.97) (xy 186.69 140.97)
+			(xy 180.34 148.59) (xy 186.69 148.59)
 		)
 		(stroke
@@
 	(wire
 		(pts
-			(xy 180.34 143.51) (xy 186.69 143.51)
+			(xy 180.34 146.05) (xy 186.69 146.05)
 		)
 		(stroke
@@
 		)
 	)
-	(label "MIDDLE"
+	(label "THUMB_2"
 		(at 120.65 54.61 180)
 		(effects
@@
 		)
 	)
-	(label "RING"
+	(label "INDEX"
 		(at 120.65 66.04 180)
 		(effects
@@
 	)
 	(label "CW"
-		(at 180.34 143.51 180)
+		(at 180.34 146.05 180)
 		(effects
 			(font
@@
 		)
 	)
-	(label "THUMB_2"
+	(label "PINKY"
 		(at 120.65 100.33 180)
 		(effects
@@
 		)
 	)
-	(label "INDEX"
+	(label "THUMB_1"
 		(at 120.65 43.18 180)
 		(effects
@@
 		)
 	)
-	(label "PINKIE"
+	(label "MIDDLE"
 		(at 120.65 77.47 180)
 		(effects
@@
 		)
 	)
-	(label "THUMB_1"
+	(label "RING"
 		(at 120.65 88.9 180)
 		(effects
@@
 	)
 	(label "DT"
-		(at 180.34 140.97 180)
+		(at 180.34 148.59 180)
 		(effects
 			(font
@@
 			)
 		)
-		(property "Footprint" "Connector_PinHeader_2.54mm:PinHeader_1x03_P2.54mm_Vertical"
+		(property "Footprint" "Connector_PinHeader_2.54mm:PinHeader_1x04_P2.54mm_Vertical"
 			(at 157.734 143.256 0)
 			(effects
@@
 	(symbol
 		(lib_id "power:GND")
-		(at 184.15 148.59 270)
+		(at 184.15 140.97 270)
+		(mirror x)
 		(unit 1)
 		(exclude_from_sim no)
@@
 		(fields_autoplaced yes)
 		(property "Reference" "#PWR27"
-			(at 177.8 148.59 0)
+			(at 177.8 140.97 0)
 			(effects
 				(font
@@
 		)
 		(property "Value" "GND"
-			(at 180.34 148.5899 90)
+			(at 180.34 140.9701 90)
 			(effects
 				(font
@@
 		)
 		(property "Footprint" ""
-			(at 184.15 148.59 0)
+			(at 184.15 140.97 0)
 			(effects
 				(font
@@
 		)
 		(property "Datasheet" ""
-			(at 184.15 148.59 0)
+			(at 184.15 140.97 0)
 			(effects
 				(font
@@
 		)
 		(property "Description" "Power symbol creates a global label with name \"GND\" , ground"
-			(at 184.15 148.59 0)
+			(at 184.15 140.97 0)
 			(effects
 				(font
@@
 	(symbol
 		(lib_id "power:+3V3")
-		(at 184.15 146.05 90)
+		(at 184.15 143.51 90)
+		(mirror x)
 		(unit 1)
 		(exclude_from_sim no)
@@
 		(fields_autoplaced yes)
 		(property "Reference" "#PWR26"
-			(at 187.96 146.05 0)
+			(at 187.96 143.51 0)
 			(effects
 				(font
@@
 		)
 		(property "Value" "+3V3"
-			(at 180.34 146.0499 90)
+			(at 180.34 143.5101 90)
 			(effects
 				(font
@@
 		)
 		(property "Footprint" ""
-			(at 184.15 146.05 0)
+			(at 184.15 143.51 0)
 			(effects
 				(font
@@
 		)
 		(property "Datasheet" ""
-			(at 184.15 146.05 0)
+			(at 184.15 143.51 0)
 			(effects
 				(font
@@
 		)
 		(property "Description" "Power symbol creates a global label with name \"+3V3\""
-			(at 184.15 146.05 0)
+			(at 184.15 143.51 0)
 			(effects
 				(font
@@
 	(symbol
 		(lib_id "Mechanical:MountingHole")
-		(at 195.58 116.84 0)
+		(at 195.58 118.11 0)
 		(unit 1)
 		(exclude_from_sim yes)
@@
 		(fields_autoplaced yes)
 		(property "Reference" "H4"
-			(at 198.12 115.5699 0)
+			(at 198.12 116.8399 0)
 			(effects
 				(font
@@
 		)
 		(property "Value" "MountingHole"
-			(at 198.12 118.1099 0)
+			(at 198.12 119.3799 0)
 			(effects
 				(font
@@
 		)
 		(property "Footprint" "MountingHole:MountingHole_5.3mm_M5"
-			(at 195.58 116.84 0)
+			(at 195.58 118.11 0)
 			(effects
 				(font
@@
 		)
 		(property "Datasheet" "~"
-			(at 195.58 116.84 0)
+			(at 195.58 118.11 0)
 			(effects
 				(font
@@
 		)
 		(property "Description" "Mounting Hole without connection"
-			(at 195.58 116.84 0)
+			(at 195.58 118.11 0)
 			(effects
 				(font
@@
 			)
 		)
-		(property "Footprint" ""
+		(property "Footprint" "Library:ESP32-WROOM-32"
 			(at 60.96 83.82 0)
 			(effects
@@
 					(size 1.27 1.27)
 				)
+				(hide yes)
 			)
 		)

Commit message: Don't clone
Parts:
- removed SW1, SW2: SW_Push, Connector_PinHeader_2.54mm:PinHeader_1x02_P2.54mm_Vertical, symbol Switch:SW_Push
Connections:
- net +3V3: no longer U3.30 (3V3)
- net CW: no longer U3.6 (G32)
- net DIR_PIN: no longer U3.28 (G15)
- net DT: no longer U3.5 (G35)
- net INDEX: no longer U3.21 (G19)
- net MIDDLE: no longer U3.20 (G21)
- net RING: no longer U3.4 (G34)
- net STEP_PIN: no longer U3.27 (G2)
- net THUMB_1: no longer U3.26 (G4)
- net THUMB_2: no longer U3.22 (G18)
- net G14: now reaches U3.11 (G14)
- net G25: now reaches U3.8 (G25)
- net EN: now reaches U3.1 (EN)
- net G27: now reaches U3.10 (G27)
- net G12: now reaches U3.12 (G12)
- net G13: now reaches U3.13 (G13)
- net 5V: now reaches U3.15 (5V)
- net G23: now reaches U3.16 (G23)
- net TX0: now reaches U3.18 (TX0)
- net RX0: now reaches U3.19 (RX0)
- net VP: now reaches U3.2 (VP)
- net D5: now reaches U3.23 (D5)
- net TX2: now reaches U3.24 (TX2)
- net RX2: now reaches U3.25 (RX2)
- net VN: now reaches U3.3 (VN)
- net G33: now reaches U3.7 (G33)
- net G26: now reaches U3.9 (G26)
- net PINKIE renamed G22
- new net 3V3: U3.30 (3V3)
- new net G15: U3.28 (G15)
- new net G18: U3.22 (G18)
- new net G19: U3.21 (G19)
- new net G2: U3.27 (G2)
- new net G21: U3.20 (G21)
- new net G32: U3.6 (G32)
- new net G34: U3.4 (G34)
- new net G35: U3.5 (G35)
- new net G4: U3.26 (G4)
- no-connect marks 17 -> 2

Commit message: Change
Parts:
- added SW1, SW2: SW_SPST, Connector_PinHeader_2.54mm:PinHeader_1x02_P2.54mm_Vertical, symbol Switch:SW_SPST
- renumbered U3 to U1, A1 to U3, Encoder1 to U4
Connections:
- net 3V3 is gone; now on net +3V3: U1.30 (3V3)
- net EN is gone; now on net +3V3: U1.1 (EN)
- net G12 is gone; now on net CW: U1.12 (G12)
- net G13 is gone; now on net DT: U1.13 (G13)
- net G18 is gone; now on net RING: U1.22 (G18)
- net G19 is gone; now on net MIDDLE: U1.21 (G19)
- net G21 is gone; now on net INDEX: U1.20 (G21)
- net G22 is gone; now on net THUMB_2: U1.17 (G22)
- net G23 is gone; now on net THUMB_1: U1.16 (G23)
- net G34 is gone; now on net STEP_PIN: U1.4 (G34)
- net G35 is gone; now on net DIR_PIN: U1.5 (G35)
- net PINKY is gone; now on net PINKIE: M6.1 (-)
- net +3V3: now also SW1.2 (B), SW2.2 (B)
- net 5V: no longer names the net of U1.15 (5V)
- net D5: no longer names the net of U1.23 (D5)
- net G14: no longer names the net of U1.11 (G14)
- net G15 renamed LIMIT_2
- net LIMIT_2: now also SW2.1 (A)
- net G2 renamed LIMIT_1
- net LIMIT_1: now also SW1.1 (A)
- net G25: no longer names the net of U1.8 (G25)
- net G26: no longer names the net of U1.9 (G26)
- net G27: no longer names the net of U1.10 (G27)
- net G32: no longer names the net of U1.6 (G32)
- net G33: no longer names the net of U1.7 (G33)
- net G4 renamed PINKIE
- net RX0: no longer names the net of U1.19 (RX0)
- net RX2: no longer names the net of U1.25 (RX2)
- net TX0: no longer names the net of U1.18 (TX0)
- net TX2: no longer names the net of U1.24 (TX2)
- net VN: no longer names the net of U1.3 (VN)
- net VP: no longer names the net of U1.2 (VP)
- no-connect marks 2 -> 16
Other:
- note added: "*20 IS NOT GROUND*"
- note added: "*PADs 31-36 DNE*"
- note added: "LIMIT SWITCHES"
- note added: "PCB Layout is EXACTLY the same as the Schematic"
- note removed: "IMPORTANT: 20 IS NOT GROUND"
- note removed: "PADs 31-36 DNE"
- moved on the sheet: C1, H1, H2, H3, H4, J1, M3, M7, U1, U2, U3, U4

Commit message: PCB V4 Done
Connections:
- net GND: no longer U1.14 (GND)
- no-connect marks 16 -> 18
Changed lines of the file:
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@@
 	)
 	(no_connect
+		(at 36.83 62.23)
+	)
+	(no_connect
+		(at 107.95 90.17)
+	)
+	(no_connect
 		(at 59.69 34.29)
 	)
@@
 					(unit 1)
 				)
-			)
-		)
-	)
-	(symbol
-		(lib_id "power:GND")
-		(at 36.83 62.23 270)
-		(mirror x)
-		(unit 1)
-		(exclude_from_sim no)
-		(in_bom yes)
-		(on_board yes)
-		(dnp no)
-		(property "Reference" "#PWR4"
-			(at 30.48 62.23 0)
-			(effects
-				(font
-					(size 1.27 1.27)
-				)
-				(hide yes)
-			)
-		)
-		(property "Value" "GND"
-			(at 33.02 62.2299 90)
-			(effects
-				(font
-					(size 1.27 1.27)
-				)
-				(justify right)
-			)
-		)
-		(property "Footprint" ""
-			(at 36.83 62.23 0)
-			(effects
-				(font
-					(size 1.27 1.27)
-				)
-				(hide yes)
-			)
-		)
-		(property "Datasheet" ""
-			(at 36.83 62.23 0)
-			(effects
-				(font
-					(size 1.27 1.27)
-				)
-				(hide yes)
-			)
-		)
-		(property "Description" "Power symbol creates a global label with name \"GND\" , ground"
-			(at 36.83 62.23 0)
-			(effects
-				(font
-					(size 1.27 1.27)
-				)
-				(hide yes)
-			)
-		)
-		(pin "1"
-		)
-		(instances
-			(project "NathanHuang_Sp25_1"
-				(path "/ab2041eb-320e-4b4d-9636-e8f50e038a2e"
-					(reference "#PWR4")
-					(unit 1)
-				)

Commit message: Changes
Parts:
- added U5: LM2596_BUCK_CONVERTER, Library:LM2596_BUCK_CONVERTER, symbol Library:LM2596_BUCK_CONVERTER
Connections:
- net +12V: now also U5.1 (Vin)
- net GND: now also U5.2 (GND), U5.3 (GND)
- new net 3.3V: U5.4 (Vout)

Commit message: Changes
Connections:
- net +12V: no longer U3.8 (VMOT)
- net GND: no longer U3.10 (MS1), U3.11 (MS2), U3.12 (MS3)
- net 3.3V renamed +3.3V
- new net 12V: U3.8 (VMOT)
- no-connect marks 18 -> 17
Changed lines of the file:
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@@
 	)
 	(junction
-		(at 130.81 121.92)
-		(diameter 0)
-		(color 0 0 0 0)
-	)
-	(junction
 		(at 82.55 132.08)
 		(diameter 0)
@@
 	)
 	(no_connect
-		(at 107.95 90.17)
-	)
-	(no_connect
 		(at 59.69 34.29)
 	)
@@
 	(wire
 		(pts
-			(xy 130.81 121.92) (xy 130.81 124.46)
-		)
-		(stroke
-			(width 0)
-			(type default)
-		)
-	)
-	(wire
-		(pts
 			(xy 33.02 57.15) (xy 36.83 57.15)
 		)
@@
 	(wire
 		(pts
+			(xy 146.05 90.17) (xy 146.05 93.98)
+		)
+		(stroke
+			(width 0)
+			(type default)
+		)
+	)
+	(wire
+		(pts
 			(xy 156.21 130.81) (xy 171.45 130.81)
 		)
@@
 		)
 	)
-	(wire
-		(pts
-			(xy 130.81 119.38) (xy 130.81 121.92)
-		)
-		(stroke
-			(width 0)
-			(type default)
-		)
-	)
 	(label "THUMB_2"
 		(at 134.62 33.02 180)
@@
 		)
 	)
-	(global_label "3.3V"
+	(global_label "7.2V"
 		(shape input)
-		(at 92.71 148.59 0)
+		(at 137.16 46.99 180)
 		(fields_autoplaced yes)
 		(effects
@@
 				(size 1.27 1.27)
 			)
-			(justify left)
+			(justify right)
 		)
 		(property "Intersheetrefs" "${INTERSHEET_REFS}"
-			(at 99.8076 148.59 0)
+			(at 130.0624 46.99 0)
 			(effects
 				(font
 					(size 1.27 1.27)
 				)
-				(justify left)
+				(justify right)
 				(hide yes)
 			)
@@
 	(global_label "7.2V"
 		(shape input)
-		(at 137.16 46.99 180)
+		(at 137.16 24.13 180)
 		(fields_autoplaced yes)
 		(effects
@@
 		)
 		(property "Intersheetrefs" "${INTERSHEET_REFS}"
-			(at 130.0624 46.99 0)
+			(at 130.0624 24.13 0)
 			(effects
 				(font
@@
 	(global_label "7.2V"
 		(shape input)
-		(at 137.16 24.13 180)
+		(at 137.16 81.28 180)
 		(fields_autoplaced yes)
 		(effects
@@
 		)
 		(property "Intersheetrefs" "${INTERSHEET_REFS}"
-			(at 130.0624 24.13 0)
+			(at 130.0624 81.28 0)
 			(effects
 				(font
@@
 		)
 	)
-	(global_label "7.2V"
+	(global_label "12V"
 		(shape input)
-		(at 137.16 81.28 180)
+		(at 146.05 90.17 90)
 		(fields_autoplaced yes)
 		(effects
@@
 				(size 1.27 1.27)
 			)
-			(justify right)
+			(justify left)
 		)
 		(property "Intersheetrefs" "${INTERSHEET_REFS}"
-			(at 130.0624 81.28 0)
+			(at 146.05 83.6772 90)
 			(effects
 				(font
 					(size 1.27 1.27)
 				)
-				(justify right)
+				(justify left)
 				(hide yes)
 			)
@@
 	(symbol
 		(lib_id "power:+12V")
-		(at 146.05 93.98 0)
-		(unit 1)
-		(exclude_from_sim no)
-		(in_bom yes)
-		(on_board yes)
-		(dnp no)
-		(property "Reference" "#PWR14"
-			(at 146.05 97.79 0)
-			(effects
-				(font
-					(size 1.27 1.27)
-				)
-				(hide yes)
-			)
-		)
-		(property "Value" "+12V"
-			(at 149.606 91.694 0)
-			(effects
-				(font
-					(size 1.27 1.27)
-				)
-			)
-		)
-		(property "Footprint" ""
-			(at 146.05 93.98 0)
-			(effects
-				(font
-					(size 1.27 1.27)
-				)
-				(hide yes)
-			)
-		)
-		(property "Datasheet" ""
-			(at 146.05 93.98 0)
-			(effects
-				(font
-					(size 1.27 1.27)
-				)
-				(hide yes)
-			)
-		)
-		(property "Description" "Power symbol creates a global label with name \"+12V\""
-			(at 146.05 93.98 0)
-			(effects
-				(font
-					(size 1.27 1.27)
-				)
-				(hide yes)
-			)
-		)
-		(pin "1"
-		)
-		(instances
-			(project ""
-				(path "/ab2041eb-320e-4b4d-9636-e8f50e038a2e"
-					(reference "#PWR14")
-					(unit 1)
-				)
-			)
-		)
-	)
-	(symbol
-		(lib_id "power:+12V")
 		(at 133.35 151.13 90)
 		(unit 1)
@@
 	(symbol
 		(lib_id "power:GND")
-		(at 130.81 121.92 270)
-		(unit 1)
-		(exclude_from_sim no)
-		(in_bom yes)
-		(on_board yes)
-		(dnp no)
-		(fields_autoplaced yes)
-		(property "Reference" "#PWR15"
-			(at 124.46 121.92 0)
-			(effects
-				(font
-					(size 1.27 1.27)
-				)
-				(hide yes)
-			)
-		)
-		(property "Value" "GND"
-			(at 127 121.9199 90)
-			(effects
-				(font
-					(size 1.27 1.27)
-				)
-				(justify right)
-			)
-		)
-		(property "Footprint" ""
-			(at 130.81 121.92 0)
-			(effects
-				(font
-					(size 1.27 1.27)
-				)
-				(hide yes)
-			)
-		)
-		(property "Datasheet" ""
-			(at 130.81 121.92 0)
-			(effects
-				(font
-					(size 1.27 1.27)
-				)
-				(hide yes)
-			)
-		)
-		(property "Description" "Power symbol creates a global label with name \"GND\" , ground"
-			(at 130.81 121.92 0)
-			(effects
-				(font
-					(size 1.27 1.27)
-				)
-				(hide yes)
-			)
-		)
-		(pin "1"
-		)
-		(instances
-			(project ""
-				(path "/ab2041eb-320e-4b4d-9636-e8f50e038a2e"
-					(reference "#PWR15")
-					(unit 1)
-				)
-			)
-		)
-	)
-	(symbol
-		(lib_id "power:GND")
 		(at 137.16 60.96 270)
 		(unit 1)
@@
 					(unit 1)
 				)
+			)
+		)
+	)
+	(symbol
+		(lib_id "power:+3.3V")
+		(at 92.71 148.59 270)
+		(unit 1)
+		(exclude_from_sim no)
+		(in_bom yes)
+		(on_board yes)
+		(dnp no)
+		(fields_autoplaced yes)
+		(property "Reference" "#PWR029"
+			(at 88.9 148.59 0)
+			(effects
+				(font
+					(size 1.27 1.27)
+				)
+				(hide yes)
+			)
+		)
+		(property "Value" "+3.3V"
+			(at 96.52 148.5899 90)
+			(effects
+				(font
+					(size 1.27 1.27)
+				)
+				(justify left)
+			)
+		)
+		(property "Footprint" ""
+			(at 92.71 148.59 0)
+			(effects
+				(font
+					(size 1.27 1.27)
+				)
+				(hide yes)
+			)
+		)
+		(property "Datasheet" ""
+			(at 92.71 148.59 0)
+			(effects
+				(font
+					(size 1.27 1.27)
+				)
+				(hide yes)
+			)
+		)
+		(property "Description" "Power symbol creates a global label with name \"+3.3V\""
+			(at 92.71 148.59 0)
+			(effects
+				(font
+					(size 1.27 1.27)
+				)
+				(hide yes)
+			)
+		)
+		(pin "1"
+		)
+		(instances
+			(project ""
+				(path "/ab2041eb-320e-4b4d-9636-e8f50e038a2e"
+					(reference "#PWR029")
+					(unit 1)
+				)
