File: Spring_2025/NathanHuang_Sp25_1/NathanHuang_Sp25_1.kicad_pcb (KiCad board)
At the start: 2 copper layers, 19 parts, among them J1 Barrel_Jack, M1 Motor_Servo, M2 Motor_Servo, M3 Motor_Servo, M4 Motor_Servo, M5 Motor_Servo, M6 Motor_Servo, M7 Stepper_Motor_bipolar, SW1 SW_Push, SW2 SW_Push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

Commit message: PCB Changes
Parts:
- moved U3 61.2 mm to (325.4, 108.4), turned to 90 degrees
- moved Encoder1 48.5 mm to (377.1, 118.0)
- moved M6 3.57 mm to (358.6, 73.0)
- moved M5 3.51 mm to (344.9, 73.0)
- moved M4 3.46 mm to (331.2, 73.0)
- moved M3 3.43 mm to (317.5, 73.0)
- moved M2 3.41 mm to (303.8, 73.0)
- moved M1 3.40 mm to (290.2, 73.0)
Connections:
- Encoder1 pad 1: GND -> /DT
- Encoder1 pad 2: +3V3 -> /CW
- Encoder1 pad 3: /CW -> +3V3
- Encoder1 pad 4: /DT -> GND
- M6 pad 1: /PINKY -> /PINKIE
- SW1 pad 1: Net-(U3-G14) -> /SW1
- SW2 pad 1: Net-(U3-G25) -> /SW2
- U3 pad 11: Net-(U3-G14) -> unconnected-(U3-G14-Pad11)
- U3 pad 12: unconnected-(U3-G12-Pad12) -> /DT
- U3 pad 13: unconnected-(U3-G13-Pad13) -> /CW
- U3 pad 16: unconnected-(U3-G23-Pad16) -> /THUMB_1
- U3 pad 17: /PINKIE -> /THUMB_2
- U3 pad 20: /MIDDLE -> /INDEX
- U3 pad 21: /INDEX -> /MIDDLE
- U3 pad 22: /THUMB_2 -> /RING
- U3 pad 26: /THUMB_1 -> /PINKIE
- U3 pad 27: /STEP_PIN -> /SW1
- U3 pad 28: /DIR_PIN -> /SW2
- U3 pad 4: /RING -> /DIR_PIN
- U3 pad 5: /DT -> /STEP_PIN
- U3 pad 6: /CW -> unconnected-(U3-G32-Pad6)
- U3 pad 8: Net-(U3-G25) -> unconnected-(U3-G25-Pad8)
Routing:
- added copper zone on B.Cu, net GND

Commit message: Change
Parts:
- removed A1: Pololu_Breakout_A4988, Module:Pololu_Breakout-16_15.2x20.3mm
- removed Encoder1: ~, Connector_PinHeader_2.54mm:PinHeader_1x04_P2.54mm_Vertical
- added U1: ESP32-WROOM-32, Library:ESP32-WROOM-32, F.Cu at (132.4, 112.6)
- added U4: ~, Connector_PinHeader_2.54mm:PinHeader_1x04_P2.54mm_Vertical, F.Cu at (178.8, 126.0)
- SW1, SW2: value SW_Push -> SW_SPST
- U3: value ESP32-WROOM-32 -> Pololu_Breakout_A4988; footprint Library:ESP32-WROOM-32 -> Module:Pololu_Breakout-16_15.2x20.3mm
- moved H2 308.3 mm to (84.7, 67.2)
- moved U3 225.3 mm to (102.2, 77.6), turned to 0 degrees
- moved H4 217.3 mm to (179.2, 137.2)
- moved U2 201.7 mm to (102.3, 124.8)
- moved SW1 200.1 mm to (183.4, 76.3), turned to 90 degrees
- moved M6 197.4 mm to (161.3, 67.0), turned to 90 degrees
- moved M5 196.3 mm to (148.7, 67.0), turned to 90 degrees
- moved J1 195.8 mm to (93.0, 119.5), turned to 0 degrees
- moved M4 195.1 mm to (136.2, 67.0), turned to 90 degrees
- moved M3 194.0 mm to (123.7, 67.0), turned to 90 degrees
- moved M2 192.8 mm to (111.1, 67.0), turned to 90 degrees
- moved M1 191.7 mm to (98.6, 67.0), turned to 90 degrees
- moved M7 191.1 mm to (83.6, 90.4)
- moved SW2 191.0 mm to (183.4, 80.2), turned to 90 degrees
- moved C1 185.2 mm to (92.1, 107.2), turned to 180 degrees
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Connections:
- M7 pad 1: Net-(A1-2B) -> Net-(U3-2B)
- M7 pad 2: Net-(A1-2A) -> Net-(M7--)
- M7 pad 3: Net-(A1-1A) -> Net-(U3-1A)
- M7 pad 4: Net-(A1-1B) -> Net-(U3-1B)
- SW1 pad 1: /SW1 -> /LIMIT_1
- SW2 pad 1: /SW2 -> /LIMIT_2
- U3 pad 1: unconnected-(U3-EN-Pad1) -> GND
- U3 pad 10: unconnected-(U3-G27-Pad10) -> GND
- U3 pad 11: unconnected-(U3-G14-Pad11) -> GND
- U3 pad 12: /DT -> GND
- U3 pad 13: /CW -> unconnected-(U3-~{RESET}-Pad13)
- U3 pad 14: GND -> unconnected-(U3-~{SLEEP}-Pad14)
- U3 pad 15: unconnected-(U3-5V-Pad15) -> /STEP_PIN
- U3 pad 16: /THUMB_1 -> /DIR_PIN
- U3 pad 2: unconnected-(U3-VP-Pad2) -> +3V3
- U3 pad 3: unconnected-(U3-VN-Pad3) -> Net-(U3-1B)
- U3 pad 4: /DIR_PIN -> Net-(U3-1A)
- U3 pad 5: /STEP_PIN -> Net-(M7--)
- U3 pad 6: unconnected-(U3-G32-Pad6) -> Net-(U3-2B)
- U3 pad 7: unconnected-(U3-G33-Pad7) -> GND
- U3 pad 8: unconnected-(U3-G25-Pad8) -> +12V
- U3 pad 9: unconnected-(U3-G26-Pad9) -> GND
Routing:
- net +3V3: track 0.00 -> 157.2 mm
- net 7.2V: track 0.00 -> 67.4 mm
- net /THUMB_1: track 0.00 -> 49.8 mm
- net /DIR_PIN: track 0.00 -> 49.7 mm
- net /STEP_PIN: track 0.00 -> 46.2 mm
- net /THUMB_2: track 0.00 -> 39.8 mm
- net /INDEX: track 0.00 -> 35.6 mm
- net /MIDDLE: track 0.00 -> 27.0 mm
- net /RING: track 0.00 -> 22.9 mm
- net /PINKIE: track 0.00 -> 21.9 mm
- net /LIMIT_1: track 0.00 -> 19.9 mm
- net Net-(U3-2B): track 0.00 -> 18.6 mm
- net Net-(U3-1A): track 0.00 -> 18.6 mm
- net Net-(M7--): track 0.00 -> 18.6 mm
- net Net-(U3-1B): track 0.00 -> 18.6 mm
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Other:
- board outline added: 122.3 x 92.8 mm
- board text added: "INDEX"
- board text added: "MIDDLE"
- board text added: "PINKIE"
- board text added: "RING"
- board text added: "THUMB_1"
- board text added: "THUMB_2"
- board text removed: "12 V OPERATION"
- board text removed: "7.2 V OPERATION"

Commit message: Gerbers ready
Parts:
- moved C1 17.6 mm to (94.1, 124.7)
- moved J1 14.6 mm to (104.7, 110.7)
- moved U4 7.29 mm to (185.9, 127.8)
- moved M3 0.63 mm to (124.3, 67.0)
- moved M4 0.50 mm to (136.7, 67.0)
- moved M5 0.38 mm to (149.1, 67.0)
- moved M2 0.32 mm to (111.4, 67.0)
- moved M6 0.25 mm to (161.5, 67.0)
Routing:
- net GND: track 13.5 -> 327.7 mm
- net 7.2V: track 67.4 -> 138.7 mm, vias 0 -> 2
- net +12V: track 12.7 -> 39.3 mm
- net +3V3: track 157.2 -> 167.1 mm
- net /DT: track 10.7 -> 18.5 mm
- net /CW: track 14.3 -> 22.1 mm
- net /MIDDLE: track 27.0 -> 30.7 mm
- net /INDEX: track 35.6 -> 36.7 mm
- removed copper zone on B.Cu, net GND
Other:
- board size 122.3 x 92.8 mm -> 112.7 x 89.7 mm
- board text added: "LIMIT SWITCH"
