File: Spring_2025/NathanHuang_Sp25_1/NathanHuang_Sp25_1.kicad_pcb (KiCad board)
At the start: 2 copper layers, 112.7 x 89.7 mm, 19 parts, among them J1 Barrel_Jack, M1 Motor_Servo, M2 Motor_Servo, M3 Motor_Servo, M4 Motor_Servo, M5 Motor_Servo, M6 Motor_Servo, M7 Stepper_Motor_bipolar, SW1 SW_SPST, SW2 SW_SPST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

Commit message: PCB V4 Done
Parts:
- moved J1 10.4 mm to (94.3, 110.8)
- moved U1 0.53 mm to (132.9, 112.7)
Connections:
- U1 pad 14: GND -> unconnected-(U1-GND-Pad14)
Routing:
- net GND: track 327.7 -> 290.1 mm
- net 7.2V: track 138.7 -> 150.2 mm
- net /MIDDLE: track 30.7 -> 27.1 mm
- net +12V: track 39.3 -> 42.3 mm
- net /INDEX: track 36.7 -> 34.9 mm
- net /DIR_PIN: track 49.7 -> 50.3 mm
- net /STEP_PIN: track 46.2 -> 46.7 mm
- net /DT: track 18.5 -> 18.0 mm
- net /CW: track 22.1 -> 21.6 mm
- net /THUMB_2: track 39.5 -> 40.0 mm
- net /THUMB_1: track 49.8 -> 50.3 mm
- net /LIMIT_1: track 19.9 -> 19.4 mm
- net /LIMIT_2: track 15.7 -> 15.2 mm
Other:
- outline, holes or cut-outs redrawn
