File: Spring_2026_Final/Hand_System_Rev_1/Hand_System_Rev_1.kicad_pcb (KiCad board)
At the start: 4 copper layers, 41 parts, among them J1 Barrel_Jack, M1 Motor_Servo, M10 Motor_Servo, M11 Motor_Servo, M2 Motor_Servo, M3 Motor_Servo, M4 Motor_Servo, M5 Motor_Servo, M6 Motor_Servo, M7 Stepper_Motor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

Commit message: Moved Buck converter down
Parts:
- moved U2 58.5 mm to (66.9, 105.0)
Routing:
- net GND: track 386.5 -> 435.2 mm
- net 12V: track 41.9 -> 66.5 mm
- net 15V: track 51.0 -> 29.7 mm
Changed lines of the file:
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@@
 	(footprint "PCB_Components:LM2596"
 		(layer "F.Cu")
-		(at 66.675 46.482)
+		(at 66.86 105)
 		(property "Reference" "U2"
 			(at 21.59 -3.81 0)
@@
 	)
 	(segment
-		(start 107.315 64.262)
-		(end 85.847 85.73)
+		(start 72.411 86.36)
+		(end 72.411 117.229)
 		(width 0.2)
 		(layer "F.Cu")
@@
 	)
 	(segment
+		(start 107.5 122.78)
+		(end 66.86 122.78)
+		(width 0.2)
+		(layer "F.Cu")
+		(net 1)
+	)
+	(segment
 		(start 183.515 126.031)
 		(end 178.181 126.031)
@@
 	)
 	(segment
+		(start 72.411 117.229)
+		(end 66.86 122.78)
+		(width 0.2)
+		(layer "F.Cu")
+		(net 1)
+	)
+	(segment
 		(start 190.119 126.031)
 		(end 195.707 126.031)
@@
 	)
 	(segment
-		(start 117.729 64.262)
-		(end 107.315 64.262)
-		(width 0.2)
-		(layer "In1.Cu")
-		(net 1)
-	)
-	(segment
-		(start 66.675 80.624)
-		(end 72.411 86.36)
+		(start 140.335 103.124)
+		(end 141.386 104.175)
 		(width 0.2)
 		(layer "In1.Cu")
@@
 	)
 	(segment
-		(start 140.335 103.124)
-		(end 141.386 104.175)
+		(start 107.5 122.78)
+		(end 135.919 122.78)
 		(width 0.2)
 		(layer "In1.Cu")
@@
 	)
 	(segment
-		(start 66.675 64.262)
-		(end 66.675 80.624)
+		(start 135.919 122.78)
+		(end 140.335 118.364)
 		(width 0.2)
 		(layer "In1.Cu")
@@
 	)
 	(segment
-		(start 77.591 57.398)
-		(end 66.675 46.482)
+		(start 83.439 86.36)
+		(end 83.947 85.852)
 		(width 0.2)
 		(layer "F.Cu")
@@
 	(segment
 		(start 77.591 86.36)
-		(end 77.591 57.398)
+		(end 83.439 86.36)
 		(width 0.2)
 		(layer "F.Cu")
@@
 	)
 	(segment
-		(start 83.439 86.36)
-		(end 83.947 85.852)
+		(start 77.591 94.269)
+		(end 66.86 105)
 		(width 0.2)
-		(layer "F.Cu")
+		(layer "In1.Cu")
 		(net 2)
 	)
 	(segment
 		(start 77.591 86.36)
-		(end 83.439 86.36)
+		(end 77.591 94.269)
 		(width 0.2)
-		(layer "F.Cu")
+		(layer "In1.Cu")
 		(net 2)
 	)
@@
 	)
 	(segment
-		(start 107.315 46.482)
-		(end 110.617 49.784)
+		(start 108.9425 76.5575)
+		(end 107.5 78)
 		(width 0.2)
 		(layer "F.Cu")
@@
 	)
 	(segment
-		(start 110.617 49.784)
+		(start 107.5 78)
+		(end 107.5 105)
+		(width 0.2)
+		(layer "F.Cu")
+		(net 37)
+	)
+	(segment
+		(start 110.617 48.883)
 		(end 110.617 76.5575)
 		(width 0.2)
@@
 	)
 	(segment
-		(start 107.315 46.482)
-		(end 117.729 46.482)
+		(start 117.729 46.482)
+		(end 113.018 46.482)
+		(width 0.2)
+		(layer "F.Cu")
+		(net 37)
+	)
+	(segment
+		(start 113.018 46.482)
+		(end 110.617 48.883)
+		(width 0.2)
+		(layer "F.Cu")
+		(net 37)
+	)
+	(segment
+		(start 110.617 76.5575)
+		(end 108.9425 76.5575)
 		(width 0.2)
 		(layer "F.Cu")
