File: Spring_2026_Final/Hand_System_Rev_1/Hand_System_Rev_1.kicad_pcb (KiCad board)
At the start: 4 copper layers, 41 parts, among them J1 Barrel_Jack, M1 Motor_Servo, M10 Motor_Servo, M11 Motor_Servo, M2 Motor_Servo, M3 Motor_Servo, M4 Motor_Servo, M5 Motor_Servo, M6 Motor_Servo, M7 Stepper_Motor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

Commit message: Finished pcb design spring 2026
Parts:
- added U6: LM2596, PCB_Components:LM2596, F.Cu at (92.7, 106.4)
- moved U5 60.8 mm to (177.8, 36.8)
- moved U2 35.4 mm to (100.6, 36.3)
- moved R14 34.0 mm to (144.6, 79.0)
- moved R15 34.0 mm to (159.5, 79.5)
- moved Q2 34.0 mm to (150.9, 79.2)
- moved C2 33.4 mm to (145.4, 133.1)
- moved R1 30.5 mm to (148.0, 66.3)
- moved H2 29.1 mm to (93.5, 35.7)
- moved H4 28.3 mm to (93.5, 135.0)
- moved J1 27.9 mm to (105.2, 90.9)
- moved C1 27.9 mm to (112.5, 90.4)
- moved R16 24.5 mm to (143.4, 128.3)
- moved Q1 23.5 mm to (153.1, 66.9)
- moved R2 23.4 mm to (160.7, 66.3)
- moved M7 16.9 mm to (148.1, 118.9)
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Routing:
- net 7.2V: track 11.8 -> 238.1 mm
- net GND: track 386.5 -> 442.6 mm
- net /STP_VG: track 91.1 -> 35.9 mm
- net 12V: track 41.9 -> 80.0 mm
- net STP_P: track 45.6 -> 16.0 mm
- net Net-(Q2-S): track 34.8 -> 61.3 mm
- net Net-(Q1-S): track 76.4 -> 97.4 mm
- net /SERVO_VG: track 15.3 -> 35.5 mm
- net /DIR_PIN: track 39.9 -> 22.6 mm
- net /MIDDLE_2: track 21.8 -> 9.54 mm
- net /RING_2: track 24.9 -> 12.6 mm
- net /RING_1: track 23.6 -> 11.3 mm
- net 15V: track 51.0 -> 63.1 mm
- net /STEP_PIN: track 41.6 -> 29.7 mm
- net /INDEX_1: track 23.7 -> 12.1 mm
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- added copper zone on B.Cu, net GND
- added copper zone on In1.Cu, net GND
Other:
- board outline added: 154.7 x 113.4 mm
- board text added: "12V to 7.2V"
- board text added: "15V to 12V"
- board text added: "7.2V to 5V"
- board text added: "Index"
- board text added: "Middle"
- board text added: "Pinkie"
- board text added: "Purdue ARC Piano Hand"
- board text added: "Ring"
- board text added: "Rotary Encoder"
- board text added: "Servo Power Switch"
- board text added: "Spring 2026 v. 1"
- board text added: "Stepper Motor"
- board text added: "Stepper Power Switch"
- board text added: "Thumb"

Commit message: finish pcb design
Parts:
- removed Q2: IRF6623, Package_DirectFET:DirectFET_ST
- added C3: 10uF, Capacitor_SMD:C_0805_2012Metric, F.Cu at (190.8, 98.9)
- added C4: 10uF, Capacitor_SMD:C_0805_2012Metric, F.Cu at (226.4, 98.8)
- added Q3: IRLZ44N, Package_TO_SOT_THT:TO-220-3_Vertical, F.Cu at (138.8, 66.5)
- added R23: 220, Resistor_SMD:R_0805_2012Metric, F.Cu at (193.3, 113.1)
- added R24: 220, Resistor_SMD:R_0805_2012Metric, F.Cu at (195.3, 113.1)
- added R25: 220, Resistor_SMD:R_0805_2012Metric, F.Cu at (197.4, 113.1)
- added R26: 220, Resistor_SMD:R_0805_2012Metric, F.Cu at (199.4, 113.1)
- added R27: 220, Resistor_SMD:R_0805_2012Metric, F.Cu at (201.4, 113.1)
- added R28: 10k, Resistor_SMD:R_0805_2012Metric, F.Cu at (194.4, 98.9)
- added R35: 10k, Resistor_SMD:R_0805_2012Metric, F.Cu at (230.0, 98.8)
- added R36: 220, Resistor_SMD:R_0805_2012Metric, F.Cu at (228.1, 113.4)
- added R37: 220, Resistor_SMD:R_0805_2012Metric, F.Cu at (230.2, 113.4)
- added R38: 220, Resistor_SMD:R_0805_2012Metric, F.Cu at (232.2, 113.4)
- added R39: 220, Resistor_SMD:R_0805_2012Metric, F.Cu at (234.2, 113.4)
- added R40: 220, Resistor_SMD:R_0805_2012Metric, F.Cu at (236.5, 113.5)
- added U7: PCA9685PW, Package_SO:TSSOP-28_4.4x9.7mm_P0.65mm, F.Cu at (194.2, 106.2)
- added U8: PCA9685PW, Package_SO:TSSOP-28_4.4x9.7mm_P0.65mm, F.Cu at (229.7, 106.4)
- C2: footprint Capacitor_SMD:C_0805_2012Metric -> Capacitor_SMD:C_1206_3216Metric
- Q1: value IRF6623 -> IRLZ44N; footprint Package_DirectFET:DirectFET_ST -> Package_TO_SOT_THT:TO-220-3_Vertical
- R15, R2: value 1k -> 100
- moved R5 42.6 mm to (190.8, 129.9)
- moved R8 35.5 mm to (213.3, 130.5)
- moved M1 34.9 mm to (212.7, 122.9)
- moved M6 33.2 mm to (200.2, 122.7)
- moved R4 33.2 mm to (188.0, 129.9)
- moved M8 28.3 mm to (218.0, 122.9)
- moved R9 26.6 mm to (216.2, 130.5)
- moved M5 26.0 mm to (195.3, 122.7)
- moved Q1 25.4 mm to (138.4, 87.6), turned to -90 degrees
- moved R3 23.5 mm to (185.4, 129.9)
- moved M9 21.1 mm to (223.3, 122.9)
- moved M4 18.8 mm to (190.2, 122.7)
- moved R10 17.0 mm to (219.0, 130.5)
- moved R15 16.9 mm to (144.4, 87.0), turned to 90 degrees
- moved R2 16.6 mm to (144.5, 70.2), turned to 90 degrees
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Connections:
- M1 pad 2: MOTOR_P -> 5V
- M10 pad 2: MOTOR_P -> 5V
- M11 pad 2: MOTOR_P -> 5V
- M8 pad 2: MOTOR_P -> 5V
- M9 pad 2: MOTOR_P -> 5V
- Q1 pad 1: Net-(Q1-D) -> Net-(Q1-G)
- Q1 pad 2: Net-(Q1-G) -> Net-(Q1-D)
- R1 pad 2: Net-(Q1-D) -> Net-(Q3-D)
- R13 pad 1: Net-(Q1-S) -> Net-(Q3-S)
- R14 pad 1: Net-(Q2-D) -> Net-(Q1-D)
- R15 pad 2: Net-(Q2-G) -> Net-(Q1-G)
- R16 pad 1: Net-(Q2-S) -> Net-(Q1-S)
- R2 pad 2: Net-(Q1-G) -> Net-(Q3-G)
- U1 pad 15: /STP_VG -> unconnected-(U1-13-Pad15)
- U1 pad 17: unconnected-(U1-D3-Pad17) -> /STP_VG
- U1 pad 23: /THUMB_1 -> unconnected-(U1-TX-Pad23)
- U1 pad 24: /THUMB_2 -> unconnected-(U1-RX-Pad24)
- U1 pad 25: /INDEX_1 -> unconnected-(U1-21-Pad25)
- U1 pad 27: /INDEX_2 -> unconnected-(U1-19-Pad27)
- U1 pad 28: /MIDDLE_1 -> unconnected-(U1-18-Pad28)
- U1 pad 29: /MIDDLE_2 -> unconnected-(U1-5-Pad29)
- U1 pad 30: /RING_1 -> unconnected-(U1-17-Pad30)
- U1 pad 31: /RING_2 -> unconnected-(U1-16-Pad31)
- U1 pad 32: /PINKIE_1 -> unconnected-(U1-4-Pad32)
- U1 pad 33: /PINKIE_2 -> /SCL_SERV
- U1 pad 34: unconnected-(U1-2-Pad34) -> /SDA_SERV
- U1 pad 35: unconnected-(U1-15-Pad35) -> /SDA_SPL
- U1 pad 36: unconnected-(U1-D1-Pad36) -> /SCL_SPL
Routing:
- net 5V: track 78.7 -> 207.2 mm
- net GND: track 442.6 -> 524.0 mm
- net Net-(Q1-S): track 97.4 -> 30.7 mm
- net Net-(Q3-S): track 0.00 -> 63.8 mm
- net Net-(Q2-S): track 61.3 -> 0.00 mm
- net /STP_VG: track 35.9 -> 86.1 mm
- net /SDA_SERV: track 0.00 -> 44.7 mm
- net /SCL_SERV: track 0.00 -> 41.3 mm
- net MOTOR_P: track 61.6 -> 28.1 mm
- net /SERVO_VG: track 35.5 -> 59.7 mm
- net /DIR_PIN: track 22.6 -> 39.9 mm
- net 7.2V: track 238.1 -> 255.2 mm
- net /SCL_SPL: track 0.00 -> 15.6 mm
- net /PINKIE_2: track 19.3 -> 4.08 mm
- net /SDA_SPL: track 0.00 -> 14.8 mm
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Other:
- board text added: "${REFERENCE}"
- board text added: "Servo Motors"
- board text added: "Splay Motors"
- board text added: "Thumb, Index, Middle, Ring, Pinkie"
- board text removed: "Index"
- board text removed: "Middle"
- board text removed: "Pinkie"
- board text removed: "Ring"
- board text removed: "Thumb"
