File: Spring_2026_Final/Hand_System_Rev_1/Hand_System_Rev_1.kicad_sch (KiCad schematic)
At the start: 41 parts, among them J1 Barrel_Jack, M1 Motor_Servo, M10 Motor_Servo, M11 Motor_Servo, M2 Motor_Servo, M3 Motor_Servo, M4 Motor_Servo, M5 Motor_Servo, M6 Motor_Servo, M7 Stepper_Motor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

Commit message: Added buck converter 12v to 5v.
Parts:
- added U6: LM2596, PCB_Components:LM2596, symbol Schematic:LM2596
Connections:
- net 12V: now also U6.1 (Vin)
- net 5V: now also U6.4 (Vout)
- net GND: now also U6.2 (GND), U6.3 (GND)
- no-connect marks 13 -> 22
Other:
- moved on the sheet: C2, M7, U3, U5
