File: Spring_2026_Final/Hand_System_Rev_1/Hand_System_Rev_1.kicad_sch (KiCad schematic)
At the start: 41 parts, among them J1 Barrel_Jack, M1 Motor_Servo, M10 Motor_Servo, M11 Motor_Servo, M2 Motor_Servo, M3 Motor_Servo, M4 Motor_Servo, M5 Motor_Servo, M6 Motor_Servo, M7 Stepper_Motor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

Commit message: Finished pcb design spring 2026
Parts:
- added U6: LM2596, PCB_Components:LM2596, symbol Schematic:LM2596
Connections:
- net 5V: now also U6.4 (Vout)
- net 7.2V: now also U6.1 (Vin)
- net GND: now also U6.2 (GND), U6.3 (GND)
- no-connect marks 13 -> 22
Other:
- moved on the sheet: C2, M7, U3, U5

Commit message: finish pcb design
Parts:
- removed Q1, Q2: IRF6623, Package_DirectFET:DirectFET_ST, symbol Transistor_FET:IRF6623
- added C3, C4: 10uF, Capacitor_SMD:C_0805_2012Metric, symbol Device:C
- added Q1, Q3: IRLZ44N, Package_TO_SOT_THT:TO-220-3_Vertical, symbol Transistor_FET:IRLZ44N
- added R23, R24, R25, R26, R27, R36, R37, R38, R39, R40: 220, Resistor_SMD:R_0805_2012Metric, symbol Device:R
- added R28, R35: 10k, Resistor_SMD:R_0805_2012Metric, symbol Device:R
- added U7, U8: PCA9685PW, Package_SO:TSSOP-28_4.4x9.7mm_P0.65mm, symbol Driver_LED:PCA9685PW
- C2: footprint Capacitor_SMD:C_0805_2012Metric -> Capacitor_SMD:C_1206_3216Metric
- R15, R2: value 1k -> 100
Connections:
- net 5V: now also M1.2 (+), M10.2 (+), M11.2 (+), M8.2 (+), M9.2 (+), C3.2, C4.2, U7.28 (VDD), U8.28 (VDD)
- net GND: now also C3.1, C4.1, R28.2, R35.2, U7.14 (VSS), U7.25 (EXTCLK), U8.14 (VSS), U8.25 (EXTCLK)
- net INDEX_1: now also R37.1; no longer U1.25 (21)
- net INDEX_2: now also R24.1; no longer U1.27 (19)
- net MIDDLE_1: now also R38.1; no longer U1.28 (18)
- net MIDDLE_2: now also R25.1; no longer U1.29 (5)
- net MOTOR_P: no longer M1.2 (+), M10.2 (+), M11.2 (+), M8.2 (+), M9.2 (+)
- net PINKIE_1: now also R40.1; no longer U1.32 (4)
- net PINKIE_2: now also R27.1; no longer U1.33 (0)
- net RING_1: now also R39.1; no longer U1.30 (17)
- net RING_2: now also R26.1; no longer U1.31 (16)
- net STP_VG: now also U1.17 (D3); no longer U1.15 (13)
- net THUMB_1: now also R36.1; no longer U1.23 (TX)
- net THUMB_2: now also R23.1; no longer U1.24 (RX)
- net at R13.1: now also Q3.3 (S)
- net at R16.1: now also Q1.3 (S)
- net at R14.1: now also Q1.2 (D)
- net at R1.2: now also Q3.2 (D)
- net at R2.2: now also Q3.1 (G)
- net at R15.2: now also Q1.1 (G)
- net SDA_SERV: now reaches U1.34 (2)
- net SDA_SERV: now also U7.27 (SDA)
- net SDA_SPL: now reaches U1.35 (15)
- net SDA_SPL: now also U8.27 (SDA)
- net SCL_SPL: now reaches U1.36 (D1)
- net SCL_SPL: now also U8.26 (SCL)
- new net: R24.2, U7.7 (LED1)
- new net: R40.2, U8.10 (LED4)
- new net: R35.1, U8.23 (~{OE})
- new net: R36.2, U8.6 (LED0)
- new net: R37.2, U8.7 (LED1)
- new net: R38.2, U8.8 (LED2)
- new net: R39.2, U8.9 (LED3)
- new net: R28.1, U7.23 (~{OE})
- new net: R23.2, U7.6 (LED0)
- new net: R27.2, U7.10 (LED4)
- new net: R26.2, U7.9 (LED3)
- new net: R25.2, U7.8 (LED2)
- new net SCL_SERV: U1.33 (0), U7.26 (SCL)
- no-connect marks 22 -> 62
Other:
- note added: "SERVO MOTOR DRIVER"
- note added: "SPLAY MOTOR DRIVER"
- moved on the sheet: C1, C2, H1, H2, H3, H4, J1, M7, U2, U3, U4, U5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
